File: VehiculeREX/VehiculeREX.kicad_sch (KiCad schematic)
At the start: 61 parts, among them CN1 ECU - CRMT, CN10 ECU Chinois, CN11 ECU Chinois, CN12 ECU Chinois, CN13 ECU Chinois, CN14 ECU Chinois, CN15 ECU Chinois, CN16 ECU Chinois, CN17 ECU Chinois, CN18 ECU Chinois, CN19 ECU Chinois, CN2 ECU - CRMT, CN20 ECU Chinois, CN21 ECU Chinois, CN22 ECU Chinois, CN23 ECU Chinois, CN24 ECU Chinois, CN26 Capteur régime moteur, CN27 Capteur régime moteur, CN28 Capteur température eau, CN29 Capteur Température Echappeme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, CN3 ECU - CRMT, CN30 Capteur température eau, CN31 Capteur température eau, CN32 Capteur Pression Température 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, CN33 Capteur Pression Température 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, CN34 Capteur Pression Température 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, CN35 Capteur Pression Température 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, CN36 Sonde Lambda UEGO, CN37 Sonde Lambda UEGO, CN38 Capteur Pression Détendeur, CN39 Capteur Pression Détendeur, CN4 ECU - CRMT, CN40 Valve Détendeur, CN41 Valve Détendeur, CN42 Solenoide Bonbonne 1, CN43 Solenoide Bonbonne 1, CN44 Solenoide Bonbonne 2, CN45 Solenoide Bonbonne 2, CN46 Bobine, CN47 Bobine, CN48 Injecteur gaz, CN49 Injecteur gaz, CN5 ECU - CRMT, CN50 Phase 1, CN51 Phase 2, CN52 Phase 3, CN57 Papillon, CN58 Papillon, CN59 REX HV PDU, CN6 ECU - CRMT, CN60 REX HV PDU, CN63 CAN 1, CN64 CAN 2, CN7 ECU Chinois, CN75 Switch Ventilateur, CN76 Switch Ventilateur, CN8 ECU Chinois, CN9 ECU Chinois, K1 BT-REX

Commit message: Je répare le git
Parts:
- removed CN40: Valve Détendeur, symbol Connector:Conn_01x02_Socket
- removed CN41: Valve Détendeur, symbol Connector:Conn_01x02_Pin
- added CN25: Valve Détendeur, symbol Connector:Conn_01x02_Socket
- added CN40: Valve Détendeur, symbol Connector:Conn_01x02_Pin
- added NT1, NT2, NT3, NT4, NT5, NT6: NetTie_2, symbol Device:NetTie_2
Connections:
- net GND-CRMT is gone; now on net CHASSIS: CN5.L1 (Pin_7), CN5.L2 (Pin_8), CN5.L3 (Pin_9), CN5.L4 (Pin_10)
- net GND-Pression-Détendeur is gone; now on net CHASSIS: CN38.1 (Pin_1)
- net GND-Solenoide-Bonbonne-1 is gone; now on net CHASSIS: CN43.2 (Pin_2)
- net GND-Solenoide-Bonbonne-2 is gone; now on net CHASSIS: CN45.2 (Pin_2)
- net GND_Bobine is gone; now on net CHASSIS: CN47.1 (Pin_1)
- net Cmd-Contact: now also NT1.2; no longer CN43.1 (Pin_1), CN45.1 (Pin_1), K1.88
- net GND-Bobine renamed CHASSIS
- net CHASSIS: now also CN25.2 (Pin_2)
- new net: K1.88, NT1.1, NT2.1, NT3.1, NT4.1, NT5.1, NT6.1
- new net 12V-LDO: NT6.2
- new net Cmd-ECU-FAN: NT4.2
- new net Cmd-Solenoide-Bonbonne-1: CN43.1 (Pin_1), NT2.2
- new net Cmd-Solenoide-Bonbonne-2: CN45.1 (Pin_1), NT3.2
- new net Cmd-Valve-Détendeur: CN25.1 (Pin_1), NT5.2
Other:
- note added: "BFI"
- note added: "BFR"
- note added: "Boitier LDO 5V"
- note added: "DCDC"
- note added: "PDU ---- Battery"
- note removed: "Power Distribution Unit"
- moved on the sheet: CN1, CN10, CN11, CN12, CN13, CN14, CN15, CN16, CN17, CN18, CN19, CN2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

Commit message: avancement schéma véhicule
Other:
- note added: "qwe"
Changed lines of the file:
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@@
+		)
+	)
+	(text "qwe"
+		(exclude_from_sim no)
+		(at 69.85 295.91 0)
+		(effects
+			(font
+				(size 1.27 1.27)
+			)
 		)
 	)

Commit message: Push AOR
Other:
- note removed: "qwe"
Changed lines of the file:
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@@
 	(wire
 		(pts
-			(xy 466.09 116.84) (xy 351.79 116.84)
+			(xy 466.09 116.84) (xy 308.61 116.84)
 		)
 		(stroke
@@
 	(wire
 		(pts
-			(xy 351.79 116.84) (xy 351.79 101.6)
+			(xy 308.61 116.84) (xy 308.61 101.6)
 		)
 		(stroke
@@
 	(wire
 		(pts
-			(xy 466.09 115.57) (xy 466.09 116.84)
+			(xy 466.09 116.84) (xy 466.09 115.57)
 		)
 		(stroke
@@
 		(effects
 			(font
-				(size 1.27 1.27)
-			)
-		)
-	)
-	(text "qwe"
-		(exclude_from_sim no)
-		(at 69.85 295.91 0)
-		(effects
-			(font
