File: VehiculeREX/VehiculeREX.kicad_sch (KiCad schematic)
At the start: 67 parts, among them CN1 ECU - CRMT, CN10 ECU Chinois, CN11 ECU Chinois, CN12 ECU Chinois, CN13 ECU Chinois, CN14 ECU Chinois, CN15 ECU Chinois, CN16 ECU Chinois, CN17 ECU Chinois, CN18 ECU Chinois, CN19 ECU Chinois, CN2 ECU - CRMT, CN20 ECU Chinois, CN21 ECU Chinois, CN22 ECU Chinois, CN23 ECU Chinois, CN24 ECU Chinois, CN25 Valve Détendeur, CN26 Capteur régime moteur, CN27 Capteur régime moteur, CN28 Capteur température eau, CN29 Capteur Température Echappeme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, CN3 ECU - CRMT, CN30 Capteur température eau, CN31 Capteur température eau, CN32 Capteur Pression Température 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, CN33 Capteur Pression Température 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, CN34 Capteur Pression Température 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, CN35 Capteur Pression Température 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, CN36 Sonde Lambda UEGO, CN37 Sonde Lambda UEGO, CN38 Capteur Pression Détendeur, CN39 Capteur Pression Détendeur, CN4 ECU - CRMT, CN40 Valve Détendeur, CN42 Solenoide Bonbonne 1, CN43 Solenoide Bonbonne 1, CN44 Solenoide Bonbonne 2, CN45 Solenoide Bonbonne 2, CN46 Bobine, CN47 Bobine, CN48 Injecteur gaz, CN49 Injecteur gaz, CN5 ECU - CRMT, CN50 Phase 1, CN51 Phase 2, CN52 Phase 3, CN57 Papillon, CN58 Papillon, CN59 REX HV PDU, CN6 ECU - CRMT, CN60 REX HV PDU, CN63 CAN 1, CN64 CAN 2, CN7 ECU Chinois, CN75 Switch Ventilateur, CN76 Switch Ventilateur, CN8 ECU Chinois, CN9 ECU Chinois, K1 BT-REX

Commit message: Ajout des bloc pour futur modif pour CRMT
Parts:
- CN27: Boitier (none) -> 2137216-1; Botier 2137216-1 -> (none)
- CN28: value Capteur température eau -> Capteur Température Echappement
Changed lines of the file:
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@@
 			)
 		)
-		(property "Value" "Capteur température eau"
+		(property "Value" "Capteur Température Echappement"
 			(at 335.28 367.03 0)
 			(effects
@@
 			)
 		)
-		(property "Botier" "2137216-1"
+		(property "Botier" ""
 			(at 321.31 269.24 0)
 			(effects
@@
 			(at 321.31 269.24 0)
 			(effects
+				(font
+					(size 1.27 1.27)
+				)
+				(hide yes)
+			)
+		)
+		(property "Boitier" "2137216-1"
+			(at 321.31 269.24 0)
+			(effects
