File: BancTest_PS1-4/BancTest_PS1-4.kicad_sch (KiCad schematic)
At the start: 13 parts, among them CN1 Starting function changeover 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, CN10 Generator input phase wires, CN11 Generator input phase wires, CN2 Indicator light socket, CN3 Choke stepper motor wires soc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, CN4 Accelerator control stepper m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, CN5 Ingniter flameout wire socket, CN6 Igniter flameout wires, CN7 144V output positive wires, CN8 144V output negative wires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

Commit message: Modif
Parts:
- removed BT1: Batterie 12V, symbol Device:Battery_Cell
Other:
- note added: "Alim commutée"
- note added: "Alim constante"
- note added: "Arret Urgence Global"
- note added: "Arret urgence Valves Bonbonnes"
- note added: "Bobine Yonda"
- note added: "ECU CRMT"
- note added: "Interco"
- note added: "Moteur"
- note added: "Papillon Yonda"
- note added: "Switch Commande Détendeur"
- note added: "Switch Contact"
- note added: "Switch Generator Enable"
- note added: "Switch ventilateur"
- note added: "Valve Détendeur"
- note added: "Valves Bonbonnes"
- note added: "WAGO+ Commuté 12V"
- note added: "WAGO+ non-commuté"
- note added: "WAGO- Commuté 12V"
- note added: "batterie 12V"
- moved on the sheet: 100A1, CN1, CN10, CN11, CN2, CN3, CN4, CN5, CN6, CN7, CN8, CN9
