File: BancTest_PS1-4/BancTest_PS1-4.kicad_sch (KiCad schematic)
At the start: 12 parts, among them CN1 Starting function changeover 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, CN10 Generator input phase wires, CN11 Generator input phase wires, CN2 Indicator light socket, CN3 Choke stepper motor wires soc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, CN4 Accelerator control stepper m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, CN5 Ingniter flameout wire socket, CN6 Igniter flameout wires, CN7 144V output positive wires, CN8 144V output negative wires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

Commit message: Ajout des bloc pour futur modif pour CRMT
Other:
- note added: "Bobine"
- note added: "Capteur Air Admission"
- note added: "Capteur Rail Injecteur"
- note added: "Capteur Régime Moteur"
- note added: "Capteur Temp Eau"
- note added: "Injecteur"
- note added: "Relai Principal"
- note added: "Sonde Lambda UEGO"
- moved on the sheet: 100A1, CN1, CN10, CN11, CN2, CN3, CN4, CN5, CN6, CN7, CN8, CN9

Commit message: push 220125
Parts:
- added CN12: Conn_01x14_Socket, symbol Connector:Conn_01x14_Socket
- added CN13: ECU, symbol Connector:Conn_01x04_Socket
- added CN14: Conn_01x28_Socket, symbol Connector:Conn_01x28_Socket
Other:
- note added: "4"
- note added: "6"
- note added: "WAGO CRMT 12V"
- note added: "WAGO CRMT GND"
- note added: "WAGO- non-commuté"

Commit message: corrections du schema du banc ps1-4
Connections:
- net at CN12.L1 (Pin_7): now also CN12.L2 (Pin_8), CN12.L3 (Pin_9), CN12.L4 (Pin_10)
- net at CN12.M1 (Pin_11): now also CN12.M2 (Pin_12), CN12.M3 (Pin_13), CN12.M4 (Pin_14)
Changed lines of the file:
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@@
 		(color 0 0 0 0)
 	)
+	(junction
+		(at 581.66 444.5)
+		(diameter 0)
+		(color 0 0 0 0)
+	)
+	(junction
+		(at 581.66 458.47)
+		(diameter 0)
+		(color 0 0 0 0)
+	)
+	(junction
+		(at 581.66 461.01)
+		(diameter 0)
+		(color 0 0 0 0)
+	)
+	(junction
+		(at 581.66 447.04)
+		(diameter 0)
+		(color 0 0 0 0)
+	)
+	(junction
+		(at 581.66 448.31)
+		(diameter 0)
+		(color 0 0 0 0)
+	)
+	(junction
+		(at 581.66 459.74)
+		(diameter 0)
+		(color 0 0 0 0)
+	)
+	(junction
+		(at 581.66 449.58)
+		(diameter 0)
+		(color 0 0 0 0)
+	)
+	(junction
+		(at 581.66 445.77)
+		(diameter 0)
+		(color 0 0 0 0)
+	)
+	(junction
+		(at 581.66 450.85)
+		(diameter 0)
+		(color 0 0 0 0)
+	)
 	(no_connect
 		(at 1021.08 251.46)
@@
 	(wire
 		(pts
-			(xy 492.76 701.04) (xy 492.76 695.96)
-		)
-		(stroke
-			(width 0.5)
-			(type default)
-			(color 255 0 0 1)
-		)
-	)
-	(wire
-		(pts
 			(xy 927.1 299.72) (xy 1008.38 299.72)
 		)
@@
 	(wire
 		(pts
+			(xy 581.66 445.77) (xy 581.66 447.04)
+		)
+		(stroke
+			(width 0.5)
+			(type default)
+			(color 255 0 0 1)
+		)
+	)
+	(wire
+		(pts
 			(xy 459.74 697.23) (xy 462.28 697.23)
 		)
@@
 	(wire
 		(pts
+			(xy 581.66 448.31) (xy 581.66 449.58)
+		)
+		(stroke
+			(width 0.5)
+			(type default)
+			(color 255 0 0 1)
+		)
+	)
+	(wire
+		(pts
 			(xy 890.27 252.73) (xy 890.27 589.28)
 		)
@@
 	(wire
 		(pts
-			(xy 388.62 429.26) (xy 497.84 429.26)
+			(xy 388.62 429.26) (xy 495.3 429.26)
 		)
 		(stroke
@@
 	(wire
 		(pts
+			(xy 492.76 698.5) (xy 495.3 698.5)
+		)
+		(stroke
+			(width 0.5)
+			(type default)
+			(color 255 0 0 1)
+		)
+	)
+	(wire
+		(pts
 			(xy 1009.65 447.04) (xy 1010.92 447.04)
 		)
@@
 	(wire
 		(pts
+			(xy 581.66 444.5) (xy 581.66 445.77)
+		)
+		(stroke
+			(width 0.5)
+			(type default)
+			(color 255 0 0 1)
+		)
+	)
+	(wire
+		(pts
 			(xy 393.7 271.78) (xy 393.7 417.83)
 		)
@@
 	(wire
 		(pts
+			(xy 581.66 457.2) (xy 581.66 458.47)
+		)
+		(stroke
+			(width 0.5)
+			(type default)
+			(color 0 0 0 1)
+		)
+	)
+	(wire
+		(pts
 			(xy 726.44 259.08) (xy 726.44 177.8)
 		)
@@
 		)
 	)
+	(wire
+		(pts
+			(xy 485.14 416.56) (xy 388.62 416.56)
+		)
+		(stroke
+			(width 0.5)
+			(type default)
+			(color 255 0 0 1)
+		)
+	)
 	(polyline
 		(pts
@@
 	(wire
 		(pts
-			(xy 497.84 429.26) (xy 497.84 701.04)
+			(xy 970.28 356.87) (xy 1033.78 356.87)
+		)
+		(stroke
+			(width 0)
+			(type default)
+			(color 0 0 0 1)
+		)
+	)
+	(wire
+		(pts
+			(xy 495.3 698.5) (xy 495.3 429.26)
 		)
 		(stroke
@@
 	(wire
 		(pts
-			(xy 970.28 356.87) (xy 1033.78 356.87)
+			(xy 497.84 477.52) (xy 497.84 701.04)
 		)
 		(stroke
 			(width 0)
 			(type default)
-			(color 0 0 0 1)
+			(color 255 255 0 1)
 		)
 	)
@@
 		)
 	)
+	(wire
+		(pts
+			(xy 497.84 477.52) (xy 1010.92 477.52)
+		)
+		(stroke
+			(width 0)
+			(type default)
+			(color 255 255 0 1)
+		)
+	)
 	(polyline
 		(pts
@@
 	(wire
 		(pts
+			(xy 581.66 449.58) (xy 581.66 450.85)
+		)
+		(stroke
+			(width 0.5)
+			(type default)
+			(color 255 0 0 1)
+		)
+	)
+	(wire
+		(pts
 			(xy 198.12 314.96) (xy 198.12 320.04)
 		)
@@
 	(wire
 		(pts
+			(xy 581.66 450.85) (xy 581.66 452.12)
+		)
+		(stroke
+			(width 0.5)
+			(type default)
+			(color 255 0 0 1)
+		)
+	)
+	(wire
+		(pts
 			(xy 474.98 698.5) (xy 474.98 701.04)
 		)
@@
 	(wire
 		(pts
+			(xy 581.66 443.23) (xy 581.66 444.5)
+		)
+		(stroke
+			(width 0.5)
+			(type default)
+			(color 255 0 0 1)
+		)
+	)
+	(wire
+		(pts
 			(xy 970.28 356.87) (xy 970.28 701.04)
 		)
@@
 	(wire
 		(pts
+			(xy 581.66 461.01) (xy 581.66 462.28)
+		)
+		(stroke
+			(width 0.5)
+			(type default)
+			(color 0 0 0 1)
+		)
+	)
+	(wire
+		(pts
 			(xy 411.48 485.14) (xy 388.62 485.14)
 		)
@@
 	(wire
 		(pts
-			(xy 388.62 424.18) (xy 939.8 424.18)
+			(xy 581.66 459.74) (xy 581.66 461.01)
 		)
 		(stroke
-			(width 0)
+			(width 0.5)
 			(type default)
-			(color 255 0 0 1)
+			(color 0 0 0 1)
 		)
 	)
 	(wire
 		(pts
-			(xy 979.17 340.36) (xy 979.17 234.95)
+			(xy 388.62 424.18) (xy 939.8 424.18)
 		)
 		(stroke
-			(width 0.762)
+			(width 0)
 			(type default)
-			(color 255 255 0 1)
+			(color 255 0 0 1)
 		)
 	)
 	(wire
 		(pts
-			(xy 492.76 695.96) (xy 485.14 695.96)
+			(xy 979.17 340.36) (xy 979.17 234.95)
 		)
 		(stroke
-			(width 0.5)
+			(width 0.762)
 			(type default)
-			(color 255 0 0 1)
+			(color 255 255 0 1)
 		)
 	)
@@
 	(wire
 		(pts
+			(xy 581.66 447.04) (xy 581.66 448.31)
+		)
+		(stroke
+			(width 0.5)
+			(type default)
+			(color 255 0 0 1)
+		)
+	)
+	(wire
+		(pts
 			(xy 1007.11 233.68) (xy 1021.08 233.68)
 		)
@@
 	(wire
 		(pts
+			(xy 908.05 474.98) (xy 1010.92 474.98)
+		)
+		(stroke
+			(width 0)
+			(type default)
+			(color 255 255 0 1)
+		)
+	)
+	(wire
+		(pts
 			(xy 502.92 233.68) (xy 502.92 177.8)
 		)
@@
 	(wire
 		(pts
-			(xy 1010.92 474.98) (xy 908.05 474.98)
+			(xy 492.76 698.5) (xy 492.76 701.04)
 		)
 		(stroke
-			(width 0)
+			(width 0.5)
 			(type default)
-			(color 255 255 0 1)
+			(color 255 0 0 1)
 		)
 	)
@@
 	(wire
 		(pts
-			(xy 485.14 695.96) (xy 485.14 701.04)
+			(xy 485.14 416.56) (xy 485.14 701.04)
 		)
 		(stroke
@@
 	(wire
 		(pts
+			(xy 581.66 458.47) (xy 581.66 459.74)
+		)
+		(stroke
+			(width 0.5)
+			(type default)
+			(color 0 0 0 1)
+		)
+	)
+	(wire
+		(pts
 			(xy 887.73 556.26) (xy 887.73 255.27)
 		)
@@
 	)
 	(rectangle
-		(start 576.58 441.96)
+		(start 576.58 440.69)
 		(end 581.66 453.39)
 		(stroke
@@
 	(label "Alim_BFI"
 		(at 236.22 350.52 90)
-		(fields_autoplaced yes)
 		(effects
 			(font
@@
 	(label "ACC_BMS"
 		(at 213.36 350.52 90)
-		(fields_autoplaced yes)
 		(effects
 			(font
@@
 	(label "CAN L"
 		(at 210.82 350.52 90)
-		(fields_autoplaced yes)
 		(effects
 			(font
@@
 	(label "GND_BFI"
 		(at 233.68 350.52 90)
-		(fields_autoplaced yes)
 		(effects
 			(font
@@
 	(label "ACC_BMS"
 		(at 127 309.88 0)
-		(fields_autoplaced yes)
 		(effects
 			(font
@@
 	(label "HV-"
 		(at 127 325.12 0)
-		(fields_autoplaced yes)
 		(effects
 			(font
@@
 	(label "Alim_BMS_cste"
 		(at 220.98 350.52 90)
-		(fields_autoplaced yes)
 		(effects
 			(font
@@
 	(label "HVIL OUT"
 		(at 127 314.96 0)
-		(fields_autoplaced yes)
 		(effects
 			(font
@@
 	(label "CAN H"
 		(at 127 299.72 0)
-		(fields_autoplaced yes)
 		(effects
 			(font
@@
 	(label "CAN L"
 		(at 127 302.26 0)
-		(fields_autoplaced yes)
 		(effects
 			(font
@@
 	(label "HVIL IN"
 		(at 127 312.42 0)
-		(fields_autoplaced yes)
 		(effects
 			(font
@@
 	(label "CAN H"
 		(at 208.28 350.52 90)
-		(fields_autoplaced yes)
 		(effects
 			(font
@@
 	(label "Alim_BMS_cste"
 		(at 127 304.8 0)
-		(fields_autoplaced yes)
 		(effects
 			(font
@@
 	(label "HV+"
 		(at 127 322.58 0)
-		(fields_autoplaced yes)
 		(effects
 			(font
@@
 	(label "GND"
 		(at 127 307.34 0)
-		(fields_autoplaced yes)
 		(effects
 			(font
